Commit message: added whole body jacobian

File: urdf/stretch.urdf (robot description, URDF)
Before this commit: robot stretch, 19 links, 18 joints
Links:
- removed link virtual_base
- removed link x_virtual_link
- removed link y_virtual_link
- removed link z_virtual_link
Joints:
- removed joint virtual_base
- removed joint x_prismatic_joint
- removed joint y_prismatic_joint
- removed joint z_revolute_joint
